Commit message: Ajout voiture Leader/Follower, modifications topics

File: src/car_description/urdf/car_master_model.urdf (robot description, URDF)
Before this commit: robot our_car_model, 7 links, 6 joints
Links:
- removed link capteur_ultrason
- link toit: mass 10 -> 100
Joints:
- removed joint chassis_to_sonar_sensor
