Commit message: Ajout capteur vitesse et modif des topics correspondants

File: src/car_description/urdf/car_follower_model.urdf (robot description, URDF)
Before this commit: robot our_car_follower_model, 7 links, 6 joints
Links:
- removed link capteur_ultrason
- added link sonar_sensor_1, mass 0.001; collision box size=0.01 0.01 0.01; visual box size=0.01 0.01 0.01
- added link sonar_sensor_2, mass 0.001; collision box size=0.01 0.01 0.01; visual box size=0.01 0.01 0.01
- added link sonar_sensor_3, mass 0.001; collision box size=0.01 0.01 0.01; visual box size=0.01 0.01 0.01
- added link speed_sensor, mass 0.001; collision box size=0.01 0.01 0.01; visual box size=0.01 0.01 0.01
Joints:
- removed joint chassis_to_sonar_sensor
- added joint chassis_to_sonar_sensor_1: type fixed, parent chassis, child sonar_sensor_1, origin xyz=1.25 0 0.41 rpy=0 0 0
- added joint chassis_to_sonar_sensor_2: type fixed, parent chassis, child sonar_sensor_2, origin xyz=1.25 -0.72 0.41 rpy=0 0 0
- added joint chassis_to_sonar_sensor_3: type fixed, parent chassis, child sonar_sensor_3, origin xyz=1.25 0.72 0.41 rpy=0 0 0
- added joint toit_to_speed_sensor: type fixed, parent toit, child speed_sensor, origin xyz=0.865 0 0.26 rpy=0 0 0

Commit message: Maj nom node et plugin

File: src/car_description/urdf/car_follower_model.urdf (robot description, URDF)
Before this commit: robot our_car_follower_model, 10 links, 9 joints
Links:
- removed link toit
- added link roof, mass 100; collision box size=1.75 1.5 0.5; visual box size=1.75 1.5 0.5
Joints:
- removed joint chassis_to_toit
- added joint chassis_to_roof: type fixed, parent chassis, child roof, origin xyz=-0.3 0 0.65
- joint toit_to_speed_sensor: parent toit -> roof
